File: camboard.sch (KiCad schematic (older format))
At the start: 30 parts, among them J1 Conn_02x05_Odd_Even, SW1 SW_Push, U1 MK82FN256VLL15, U2 Serial-Flash, U3 Serial-Flash

Commit message: Schematic capture complete
Parts:
- removed R8, R9: 4.7K, Resistor_SMD:R_0402_1005Metric, symbol Device:R_Small_US
- removed U3: Serial-Flash, symbol symbols:Serial-Flash
- added BT1, BT2, BT3, BT4: AAA Cell, symbol Device:Battery_Cell
- added C16: 4.7uF, Capacitor_SMD:C_0805_2012Metric, symbol Device:C_Small
- added C17: 0.1uF, Capacitor_SMD:C_0402_1005Metric, symbol Device:C_Small
- added D1: LED, Resistor_SMD:R_0603_1608Metric_Pad1.05x0.95mm_HandSolder, symbol Device:LED
- added D2, D3: D_Schottky, symbol Device:D_Schottky
- added J2: Conn_02x25_Counter_Clockwise, Connector_FFC-FPC:Hirose_FH12-50S-0.5SH_1x50-1MP_P0.50mm_Horizontal, symbol Connector_Generic:Conn_02x25_Counter_Clockwise
- added J3: Conn_02x12_Counter_Clockwise, Connector_FFC-FPC:Hirose_FH12-24S-0.5SH_1x24-1MP_P0.50mm_Horizontal, symbol Connector_Generic:Conn_02x12_Counter_Clockwise
- added L1: 4.7uH, symbol Device:L_Small
- added R10, R12, R14: DNP, Resistor_SMD:R_0402_1005Metric, symbol Device:R_Small_US
- added R11, R13, R15, R16, R17, R18: 4.7K, Resistor_SMD:R_0402_1005Metric, symbol Device:R_Small_US
- added R19: 2R / 250mW / 1%, Resistor_SMD:R_0805_2012Metric_Pad1.15x1.40mm_HandSolder, symbol Device:R_Small_US
- added R20: 180, Resistor_SMD:R_0402_1005Metric, symbol Device:R_Small_US
- added SW3: SW_SPST, symbol Switch:SW_SPST
- added TP4, TP5, TP6, TP7, TP8, TP9: TestPoint, TestPoint:TestPoint_Pad_D1.5mm, symbol Connector:TestPoint
- added U3: TPS61166, footprints:WSON-10_2.5x2.5mm_P0.5mm, symbol symbols:TPS61166
- added Y1: 32.768KHz, symbol Device:Crystal
- C15: value 0.1uF -> 4.7uF; footprint Capacitor_SMD:C_0402_1005Metric -> Capacitor_SMD:C_0805_2012Metric
Connections:
- net labels added: BKLT_A, BKLT_EN, BKLT_K, BKLT_PWM, CAM_D0, CAM_D1, CAM_D2, CAM_D3, CAM_D4, CAM_D5, CAM_D6, CAM_D7, CAM_D8, CAM_D9, CAM_HREF, CAM_PCLK, CAM_PWRDN, CAM_RST_b, CAM_SIO_C, CAM_SIO_D, CAM_VSYNC, CAM_XCLK1, CTP_INT, CTP_RST_b, CTP_SCL, CTP_SDA, DISP_CSX, DISP_DB0, DISP_DB1, DISP_DB10, DISP_DB11, DISP_DB12, DISP_DB13, DISP_DB14, DISP_DB15, DISP_DB2, DISP_DB3, DISP_DB4, DISP_DB5, DISP_DB6, DISP_DB7, DISP_DB8, DISP_DB9, DISP_DCX, DISP_IM0, DISP_IM1, DISP_IM2, DISP_RDX, DISP_RESET_b, DISP_WRX, VBAT, VDD_REGIN, VREF
- net labels removed: QSPIB_CLK, QSPIB_CS_b, QSPIB_D0, QSPIB_D1, QSPIB_D2, QSPIB_D3
- wire segments 97 -> 247
- no-connect marks 0 -> 19
Other:
- note added: "16bit DBI Type B Display Interface\nfor ILI9488 Display Controller"
- note added: "24-pin FPC Camera Interface for\nOV5xxx - OV7xxx series cameras"
- note added: "Backlight Driver"
- note added: "Batteries"
- note added: "Power Switch"
- moved on the sheet: C10, C11, C14, R6, R7, U2

Commit message: Add serial port and USB connectors
Parts:
- added D4, D5, D6: D_Schottky, symbol Device:D_Schottky
- added J4: USB_B_Micro, symbol Connector:USB_B_Micro
- added J5: Conn_01x03, symbol Connector_Generic:Conn_01x03
- added R21, R22, R23: 33, Resistor_SMD:R_0402_1005Metric, symbol Device:R_Small_US
- added R24, R25: 4.7K, Resistor_SMD:R_0402_1005Metric, symbol Device:R_Small_US
Connections:
- net labels added: UART_RX, UART_TX, USB_D+, USB_D-, USB_OTG_ID
- net labels removed: VDD_REG
- wire segments 247 -> 267
- no-connect marks 19 -> 14
Other:
- note added: "Micro USB"
- note added: "UART Serial Interface"

Commit message: Layout complete
Parts:
- removed BT4: AAA Cell, symbol Device:Battery_Cell
- removed D2: D_Schottky, symbol Device:D_Schottky
- removed R17: 4.7K, Resistor_SMD:R_0402_1005Metric, symbol Device:R_Small_US
- removed TP8, TP9: TestPoint, TestPoint:TestPoint_Pad_D1.5mm, symbol Connector:TestPoint
- removed U3: TPS61166, footprints:WSON-10_2.5x2.5mm_P0.5mm, symbol symbols:TPS61166
- added C18, C19: 0.1uF, Capacitor_SMD:C_0402_1005Metric, symbol Device:C_Small
- added D0, D7: D_Schottky, Diode_SMD:D_SOT-23_ANK, symbol Device:D_Schottky
- added U3: TPS61169, footprints:SC70-5, symbol symbols:TPS61169
- BT1, BT2, BT3: value AAA Cell -> Battery_Cell; footprint (none) -> footprints:BAT_AAA_Keystone_55_56; MFR (none) -> Keystone Electronics; MPN (none) -> 55
- C1, C10, C14, C17, C2, C3, C4, C5, C6, C7, C8, C9: MFR (none) -> Kemet; MPN (none) -> C0402C104K4RAC7411
- C11, C12, C13: MFR (none) -> TDK; MPN (none) -> C1005X5R1V105K050BE
- C15: MFR (none) -> Kemet; MPN (none) -> C1206C475K4NACAUTO
- C16: value 4.7uF -> 1uF
- D1: MFR (none) -> ROHM; MPN (none) -> SML-D12P8WT86C
- D2: renamed from D3; footprint (none) -> Diode_SMD:D_SOT-23_ANK; MFR (none) -> ROHM; MPN (none) -> BAT54SHMFHT116
- D4, D5, D6: footprint (none) -> Diode_SMD:D_SOT-23_ANK; MFR (none) -> ROHM; MPN (none) -> BAT54SHMFHT116
- J2: footprint Connector_FFC-FPC:Hirose_FH12-50S-0.5SH_1x50-1MP_P0.50mm_Horizontal -> footprints:LCD_ER-TFT035-6; MFR (none) -> Molex; MPN (none) -> 541045031
- J3: footprint Connector_FFC-FPC:Hirose_FH12-24S-0.5SH_1x24-1MP_P0.50mm_Horizontal -> footprints:OV5640-5MP-Camera; MFR (none) -> Wurth; MPN (none) -> 687124183722
- J4: footprint (none) -> Connector_USB:USB_Micro-B_Molex_47346-0001; MFR (none) -> Molex; MPN (none) -> 47346-0001
- J5: footprint (none) -> Connector_PinHeader_2.54mm:PinHeader_1x03_P2.54mm_Vertical
- L1: footprint (none) -> Inductor_SMD:L_0805_2012Metric_Pad1.15x1.40mm_HandSolder; MFR (none) -> TDK; MPN (none) -> KLZ2012MHR4R7WTD25
- R11, R13, R15, R16, R18, R24, R25, R6, R7: MFR (none) -> Vishay; MPN (none) -> CRCW04024K70JNEDC
- R19: value 2R / 250mW / 1% -> 2R / 1%; MFR (none) -> Panasonic; MPN (none) -> ERJ-6DQJ2R0V
- R2, R3: MFR (none) -> ROHM; MPN (none) -> SFR01MZPF1002
- R20: value 180 -> 91; MFR (none) -> Panasonic; MPN (none) -> ERJ-2RKF91R0X
- R21, R22, R23: MFR (none) -> Vishay; MPN (none) -> CRCW040233R0JNEDC
- SW1: footprint Button_Switch_THT:SW_PUSH_6mm -> Switches:TACTILE_SWITCH_SMD_6.0X3.5MM; MFR (none) -> E-Switch; MPN (none) -> TL3302AF180QG
- SW3: footprint (none) -> Switches:SWITCH_SPST_SMD_A; MFR (none) -> C&K; MPN (none) -> PCM13SMTR
- TP1, TP2, TP3: footprint TestPoint:TestPoint_THTPad_D2.0mm_Drill1.0mm -> TestPoint:TestPoint_Pad_D1.5mm
- U1: MFR (none) -> NXP; MPN (none) -> MK82FN256VLL15
- U2: footprint (none) -> footprints:WSON8-6X5MM; MFR (none) -> ISSI; MPN (none) -> IS25WP016D-JKLE
- Y1: footprint (none) -> Crystal:Crystal_SMD_EuroQuartz_EQ161-2Pin_3.2x1.5mm; MFR (none) -> ECS; MPN (none) -> ECS-.327-12.5-34B-TR
Connections:
- net labels removed: BKLT_EN
- wire segments 267 -> 264
Other:
- moved on the sheet: C10, C11, C15, C16, D2, L1, R18, R19, TP7

Commit message: Update switch MPN
Parts:
- SW3: MPN PCM13SMTR -> PCM12SMTR
Changed lines of the file:
@@
 EESchema Schematic File Version 4
 LIBS:camboard-cache
-EELAYER 26 0
+EELAYER 29 0
 EELAYER END
 $Descr A4 11693 8268
@@
 F 3 "" H 7050 4750 50  0001 C CNN
 F 4 "C&K" H 7050 4750 50  0001 C CNN "MFR"
-F 5 "PCM13SMTR" H 7050 4750 50  0001 C CNN "MPN"
+F 5 "PCM12SMTR" H 7050 4750 50  0001 C CNN "MPN"
 	1    7050 4750
 	1    0    0    -1

Commit message: Update 4.7uF MPN
Parts:
- C15: MPN C1206C475K4NACAUTO -> 0805B475K6R3CT
Changed lines of the file:
@@
 F 3 "~" H 6900 1050 50  0001 C CNN
 F 4 "Kemet" H 0   0   50  0001 C CNN "MFR"
-F 5 "C1206C475K4NACAUTO" H 0   0   50  0001 C CNN "MPN"
+F 5 "0805B475K6R3CT" H 0   0   50  0001 C CNN "MPN"
 	1    6900 1050
 	1    0    0    -1

Commit message: Update MPN for reset button
Parts:
- C15: MFR Kemet -> Walsin
- SW1: MFR E-Switch -> C&K; MPN TL3302AF180QG -> KSR251GLFS
Changed lines of the file:
@@
 F 2 "Switches:TACTILE_SWITCH_SMD_6.0X3.5MM" H 2000 7450 50  0001 C CNN
 F 3 "" H 2000 7450 50  0001 C CNN
-F 4 "E-Switch" H 0   0   50  0001 C CNN "MFR"
-F 5 "TL3302AF180QG" H 0   0   50  0001 C CNN "MPN"
+F 4 "C&K" H 0   0   50  0001 C CNN "MFR"
+F 5 "KSR251GLFS" H 0   0   50  0001 C CNN "MPN"
 	1    2000 7250
 	0    1    1    0
@@
 F 2 "Capacitor_SMD:C_0805_2012Metric" H 6900 1050 50  0001 C CNN
 F 3 "~" H 6900 1050 50  0001 C CNN
-F 4 "Kemet" H 0   0   50  0001 C CNN "MFR"
+F 4 "Walsin" H 0   0   50  0001 C CNN "MFR"
 F 5 "0805B475K6R3CT" H 0   0   50  0001 C CNN "MPN"
 	1    6900 1050

Commit message: Power LCD backlight from VREG_IN, instead of 3.3 rail
Connections:
- wire segments 264 -> 265
Changed lines of the file:
@@
 Wire Wire Line
 	7450 950  7250 950
-$Comp
-L power:+3.3V #PWR0135
-U 1 1 5C79CEEB
-P 6900 950
-F 0 "#PWR0135" H 6900 800 50  0001 C CNN
-F 1 "+3.3V" H 6915 1123 50  0000 C CNN
-F 2 "" H 6900 950 50  0001 C CNN
-F 3 "" H 6900 950 50  0001 C CNN
-	1    6900 950
-	1    0    0    -1
-$EndComp
 Connection ~ 7250 950
 $Comp
@@
 $EndComp
 Wire Wire Line
-	6900 950  7250 950
-Connection ~ 6900 950
+	6600 950  6900 950
 $Comp
 L Device:C_Small C16
@@
 $EndComp
 NoConn ~ 1300 4800
+Connection ~ 6900 950
+Wire Wire Line
+	6900 950  7250 950
+Text Label 6600 950  0    50   ~ 0
+VDD_REGIN
 $EndSCHEMATC
